File: KiCAD files/USB-hub-daughterboard.kicad_pcb (KiCad board)
At the start: 2 copper layers, 56 parts, among them J1 TYPE-C-31-M12_13, J2 USB_A, J3 USB_A, J4 SM04B-SRSS-TB(LF)(SN), J5 SM04B-SRSS-TB(LF)(SN), U1 USBLC6-2SC6, U2 AP2112K-3.3, U3 USB2514B_Bi, U4 USBLC6-2SC6, U5 USBLC6-2SC6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

Commit message: More layout work
Parts:
- added D1: SMF9.0CA, AcheronComponents:D_SOD-123_Bidirectional, F.Cu at (-7.80, 6.90)
- moved C7 72.2 mm to (14.8, 14.6), turned to 90 degrees
- moved C4 56.5 mm to (1.13, 15.9)
- moved C3 49.2 mm to (-2.39, 18.9), turned to -90 degrees
- moved C8 49.1 mm to (15.6, 17.2)
- moved C6 48.5 mm to (5.62, 19.9), turned to -90 degrees
- moved C5 27.4 mm to (-1.77, -19.8)
- moved C11 27.4 mm to (-1.68, -13.5)
- moved C9 27.4 mm to (-1.77, -11.7)
- moved U2 27.4 mm to (-1.68, -16.5)
- moved D2 26.2 mm to (1.40, -13.1)
- moved F1 26.0 mm to (1.40, -17.9)
- moved R2 12.2 mm to (-3.08, 5.66)
- moved U7 7.92 mm to (27.9, 14.5), turned to 90 degrees
- moved H2 6.32 mm to (-34.0, 26.0)
- moved H3 6.32 mm to (34.0, 26.0)
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Connections:
- U4 pad 2: GNDPWR -> GND
- U5 pad 2: GNDPWR -> GND
Routing:
- net D1P+: track 0.00 -> 36.0 mm
- net D2P+: track 0.00 -> 35.9 mm
- net D1P-: track 0.00 -> 35.0 mm
- net D2P-: track 0.00 -> 34.8 mm
- net +3V3: track 6.26 -> 28.5 mm, vias 0 -> 3
- net D4P-: track 0.00 -> 21.2 mm
- net D4P+: track 0.00 -> 20.9 mm
- net GND: track 2.63 -> 22.0 mm, vias 0 -> 11
- net VCC: track 10.1 -> 29.5 mm
- net Net-(C3-Pad2): track 0.00 -> 15.8 mm
- net D3+: track 0.00 -> 14.7 mm
- net D3-: track 0.00 -> 14.4 mm
- net D1+: track 0.00 -> 14.3 mm
- net D1-: track 0.00 -> 13.1 mm
- net D3P-: track 0.00 -> 12.0 mm
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- added copper zone on B.Cu, net GND
- added copper zone on F.Cu, net GND
Other:
- board outline added: 86 x 33 mm

Commit message: Initial revision
Parts:
- removed C14, C15, C16, C17: 100nF, Capacitor_SMD:C_0603_1608Metric_Pad1.05x0.95mm_HandSolder
- moved C19 81.7 mm to (-27.8, 21.7), turned to 180 degrees
- moved C18 71.1 mm to (-22.7, 13.7), turned to 180 degrees
- moved R6 69.8 mm to (6.47, 9.82)
- moved R4 68.4 mm to (3.92, 18.3), turned to 90 degrees
- moved C20 62.3 mm to (35.1, 13.3), turned to 180 degrees
- moved C12 61.3 mm to (12.2, 11.5)
- moved R5 57.0 mm to (2.40, 23.1)
- moved R3 54.0 mm to (-14.1, 12.6), turned to -90 degrees
- moved R7 50.4 mm to (9.45, 10.3), turned to -90 degrees
- moved C21 48.5 mm to (30.1, 21.5), turned to 180 degrees
- moved C10 45.8 mm to (5.72, 12.6), turned to 90 degrees
- moved C13 40.9 mm to (10.9, 23.7), turned to -90 degrees
- moved C2 39.2 mm to (18.4, 16.0), turned to -90 degrees
- moved C5 33.9 mm to (-11.8, 12.6), turned to -90 degrees
- moved U2 31.6 mm to (-8.87, 14.2)
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Connections:
- U6 pad 2: GNDPWR -> GND
- U7 pad 2: GNDPWR -> GND
Routing:
- net VCC: track 29.5 -> 173.6 mm, vias 0 -> 4
- net +3V3: track 28.5 -> 79.1 mm, vias 3 -> 7
- net GND: track 22.0 -> 5.43 mm, vias 11 -> 29
- net Net-(R5-Pad2): track 0.00 -> 8.63 mm, vias 0 -> 2
- net Net-(R6-Pad2): track 0.00 -> 4.28 mm, vias 0 -> 2
- net D1P-: track 35.0 -> 36.9 mm
- net Net-(C4-Pad2): track 7.45 -> 9.25 mm
- net Net-(R7-Pad2): track 0.00 -> 1.77 mm
- net D2P-: track 34.8 -> 36.0 mm
- net D2P+: track 35.9 -> 37.0 mm
- net D3-: track 14.4 -> 15.5 mm
- net Net-(C3-Pad2): track 15.8 -> 16.6 mm
- net D3+: track 14.7 -> 15.5 mm
- net DUP-: track 8.10 -> 8.73 mm
- net GNDPWR: vias 0 -> 1
- added copper zone on B.Cu, net +3V3
- added copper zone on F.Cu, net +3V3
- added copper zone on B.Cu, net VCC
- added copper zone on F.Cu, net VCC
