File: KiCAD files/USB-hub-daughterboard.kicad_sch (KiCad schematic)
At the start: 51 parts

Commit message: Work in progress updates
Parts:
- removed D?: 1N4007, Diode_THT:D_DO-41_SOD81_P10.16mm_Horizontal, symbol Diode:1N4007
- removed U? (x3): TPD4E05U06DQAR, Package_SON:USON-10_2.5x1.0mm_P0.5mm, symbol AcheronLib:TPD4E05U06DQAR
- removed U?: TLV1117-33, symbol Regulator_Linear:TLV1117-33
- removed Y?: 24MHz, symbol Device:Crystal
- added D2: 1N5819, Diode_SMD:D_SOD-123, symbol Diode:1N5819
- added H10, H9: MountingHole, MountingHole:MountingHole_3.2mm_M3_ISO7380, symbol Mechanical:MountingHole
- added H11, H12: MountingHole, MountingHole:MountingHole_2.2mm_M2_ISO7380, symbol Mechanical:MountingHole
- added U1, U4, U5, U6, U7: USBLC6-2SC6, Package_TO_SOT_SMD:SOT-23-6, symbol Power_Protection:USBLC6-2SC6
- added U2: AP2112K-3.3, Package_TO_SOT_SMD:SOT-23-5, symbol Regulator_Linear:AP2112K-3.3
- added Y1: Crystal_GND24, Crystal:Crystal_SMD_3225-4Pin_3.2x2.5mm_HandSoldering, symbol Device:Crystal_GND24
- C1, C2: renamed from C?; footprint (none) -> Capacitor_SMD:C_0805_2012Metric_Pad1.15x1.40mm_HandSolder
- C10, C11, C12, C13, C14, C15, C16, C17, C3, C4, C6, C7, C8: renamed from C?; footprint (none) -> Capacitor_SMD:C_0603_1608Metric_Pad1.05x0.95mm_HandSolder
- C18, C19, C20, C21: renamed from C?; value 22u -> 10u; footprint (none) -> Capacitor_SMD:C_0805_2012Metric_Pad1.15x1.40mm_HandSolder
- C5: renamed from C?; value 22u -> 1u; footprint (none) -> Capacitor_SMD:C_0805_2012Metric_Pad1.15x1.40mm_HandSolder
- C9: renamed from C?; value 10u -> 1u; footprint (none) -> Capacitor_SMD:C_0805_2012Metric_Pad1.15x1.40mm_HandSolder
- H1, H2, H3: renamed from H?; footprint (none) -> MountingHole:MountingHole_3.2mm_M3_ISO7380
- H4: renamed from H?; footprint (none) -> MountingHole:MountingHole_3.2mm_M3_ISO7380_Pad
- H5: renamed from H?; footprint (none) -> MountingHole:MountingHole_2.2mm_M2_ISO7380_Pad
- H6, H7, H8: renamed from H?; footprint (none) -> MountingHole:MountingHole_2.2mm_M2_ISO7380
- J1: renamed from J?; footprint acheronConnectors:TYPE-C-31-M-12 -> AcheronConnectors:TYPE-C-31-M-12
- J2, J3: renamed from J?; footprint (none) -> Connector_USB:USB_A_Molex_67643_Horizontal
- J4, J5: renamed from J?; footprint random-keyboard-parts:JST-SR-4 -> AcheronConnectors:SM04B-SRSS-TB(LF)(SN)
- R1, R2: renamed from R?; footprint Resistors_SMD:R_0603 -> Resistor_SMD:R_0805_2012Metric_Pad1.15x1.40mm_HandSolder
- R3, R4, R5, R6, R7: renamed from R?; footprint (none) -> Resistor_SMD:R_0805_2012Metric_Pad1.15x1.40mm_HandSolder
- gave numbers to parts that had none: 4
Connections:
- net +3V3: now also D2.2 (A), U2.5 (VOUT)
- net D1+: now also U4.6 (I/O1); no longer U3.2 (USBDP_DN1/PRT_DIS_P1)
- net D1-: now also U4.4 (I/O2); no longer U3.1 (USBDM_DN1/PRT_DIS_M1)
- net D2+: now also J5.3 (Pin_3), U5.6 (I/O1); no longer J3.3 (D+), U3.4 (USBDP_DN2/PRT_DIS_P2)
- net D2-: now also J5.2 (Pin_2), U5.4 (I/O2); no longer J3.2 (D-), U3.3 (USBDM_DN2/PRT_DIS_M2)
- net D3+: now also U6.6 (I/O1); no longer U3.7 (USBDP_DN3/PRT_DIS_P3)
- net D3-: now also U6.4 (I/O2); no longer U3.6 (USBDM_DN3/PRT_DIS_M3)
- net D4+: now also J3.3 (D+), U7.6 (I/O1); no longer J5.3 (Pin_3), U3.9 (USBDP_DN4/PRT_DIS_P4)
- net D4-: now also J3.2 (D-), U7.4 (I/O2); no longer J5.2 (Pin_2), U3.8 (USBDM_DN4/PRT_DIS_M4)
- net GND: now also L1.1, U2.2 (GND), Y1.2, Y1.4
- net GNDPWR: now also U1.2 (GND), U4.2 (GND), U5.2 (GND), U6.2 (GND), U7.2 (GND)
- net VBUS: now also J1.B4 (VBUS), U1.5 (VBUS)
- net VCC: now also D2.1 (K), U2.1 (VIN), U2.3 (EN), U4.5 (VBUS), U5.5 (VBUS), U6.5 (VBUS), U7.5 (VBUS)
- net at C4.2, R4.2, U3.32 (XTALOUT): now also Y1.3
- net at C3.2, R4.1, U3.33 (XTALIN/CLKIN): now also Y1.1
- net DAU+ renamed DUP+
- net DUP+: now also U1.3 (I/O2); no longer U3.31 (USBDP_UP)
- net DAU- renamed DUP-
- net DUP-: now also U1.1 (I/O1); no longer U3.30 (USBDM_UP)
- new net D1P+: U3.2 (USBDP_DN1/PRT_DIS_P1), U4.1 (I/O1)
- new net D1P-: U3.1 (USBDM_DN1/PRT_DIS_M1), U4.3 (I/O2)
- new net D2P+: U3.4 (USBDP_DN2/PRT_DIS_P2), U5.1 (I/O1)
- new net D2P-: U3.3 (USBDM_DN2/PRT_DIS_M2), U5.3 (I/O2)
- new net D3P+: U3.7 (USBDP_DN3/PRT_DIS_P3), U6.1 (I/O1)
- new net D3P-: U3.6 (USBDM_DN3/PRT_DIS_M3), U6.3 (I/O2)
- new net D4P+: U3.9 (USBDP_DN4/PRT_DIS_P4), U7.1 (I/O1)
- new net D4P-: U3.8 (USBDM_DN4/PRT_DIS_M4), U7.3 (I/O2)
- new net DUPP+: U1.4 (I/O2), U3.31 (USBDP_UP)
- new net DUPP-: U1.6 (I/O1), U3.30 (USBDM_UP)
Other:
- moved on the sheet: C3, C4, H1, H2, H3, H4, H5, H6, H7, H8

Commit message: More layout work
Parts:
- D1: footprint acheron_Components:D_SOD-123_Bidirectional -> AcheronComponents:D_SOD-123_Bidirectional
Connections:
- net GND: now also U4.2 (GND), U5.2 (GND)
- net GNDPWR: no longer U4.2 (GND), U5.2 (GND)
Changed lines of the file:
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@@
+    (stroke (width 0) (type solid) (color 0 0 0 0))
+  )
+  (wire (pts (xy 180.975 130.175) (xy 180.975 128.905))
+    (stroke (width 0) (type solid) (color 0 0 0 0))
+  )
+  (wire (pts (xy 180.975 130.175) (xy 197.485 130.175))
     (stroke (width 0) (type solid) (color 0 0 0 0))
   )
@@
     (stroke (width 0) (type solid) (color 0 0 0 0))
   )
-  (wire (pts (xy 186.055 128.905) (xy 186.055 130.175))
-    (stroke (width 0) (type solid) (color 0 0 0 0))
-  )
   (wire (pts (xy 187.325 40.005) (xy 197.485 40.005))
     (stroke (width 0) (type solid) (color 0 0 0 0))
@@
   )
   (wire (pts (xy 197.485 117.475) (xy 191.135 117.475))
-    (stroke (width 0) (type solid) (color 0 0 0 0))
-  )
-  (wire (pts (xy 197.485 130.175) (xy 186.055 130.175))
     (stroke (width 0) (type solid) (color 0 0 0 0))
   )
@@
     (pin "1")
   )
+  (symbol (lib_id "power:+3.3V") (at 180.975 128.905 0) (unit 1)
+    (in_bom yes) (on_board yes)
+    (property "Reference" "#PWR0139" (id 0) (at 180.975 132.715 0)
+      (effects (font (size 1.27 1.27)) hide)
+    )
+    (property "Value" "+3.3V" (id 1) (at 175.895 128.27 0))
+    (property "Footprint" "" (id 2) (at 180.975 128.905 0)
+      (effects (font (size 1.27 1.27)) hide)
+    )
+    (property "Datasheet" "" (id 3) (at 180.975 128.905 0)
+      (effects (font (size 1.27 1.27)) hide)
+    )
+    (pin "1")
+  )
   (symbol (lib_id "power:+3.3V") (at 183.515 24.13 0) (unit 1)
     (in_bom yes) (on_board yes)
@@
     (pin "1")
   )
-  (symbol (lib_id "power:+3.3V") (at 186.055 128.905 0) (unit 1)
-    (in_bom yes) (on_board yes)
-    (property "Reference" "#PWR0139" (id 0) (at 186.055 132.715 0)
-      (effects (font (size 1.27 1.27)) hide)
-    )
-    (property "Value" "+3.3V" (id 1) (at 180.975 128.27 0))
-    (property "Footprint" "" (id 2) (at 186.055 128.905 0)
-      (effects (font (size 1.27 1.27)) hide)
-    )
-    (property "Datasheet" "" (id 3) (at 186.055 128.905 0)
-      (effects (font (size 1.27 1.27)) hide)
-    )
-    (pin "1")
-  )
   (symbol (lib_id "power:+3.3V") (at 191.135 115.57 0) (unit 1)
     (in_bom yes) (on_board yes)
@@
     (pin "1")
   )
-  (symbol (lib_id "power:GNDPWR") (at 280.67 45.72 0) (unit 1)
-    (in_bom yes) (on_board yes)
-    (property "Reference" "#PWR0165" (id 0) (at 280.67 50.8 0)
-      (effects (font (size 1.27 1.27)) hide)
-    )
-    (property "Value" "GNDPWR" (id 1) (at 280.67 48.26 0)
-      (effects (font (size 0.381 0.381)))
-    )
-    (property "Footprint" "" (id 2) (at 280.67 46.99 0)
-      (effects (font (size 1.27 1.27)) hide)
-    )
-    (property "Datasheet" "" (id 3) (at 280.67 46.99 0)
-      (effects (font (size 1.27 1.27)) hide)
-    )
-    (pin "1")
-  )
-  (symbol (lib_id "power:GNDPWR") (at 280.67 76.2 0) (unit 1)
-    (in_bom yes) (on_board yes)
-    (property "Reference" "#PWR0122" (id 0) (at 280.67 81.28 0)
-      (effects (font (size 1.27 1.27)) hide)
-    )
-    (property "Value" "GNDPWR" (id 1) (at 280.67 78.74 0)
-      (effects (font (size 0.381 0.381)))
-    )
-    (property "Footprint" "" (id 2) (at 280.67 77.47 0)
-      (effects (font (size 1.27 1.27)) hide)
-    )
-    (property "Datasheet" "" (id 3) (at 280.67 77.47 0)
-      (effects (font (size 1.27 1.27)) hide)
-    )
-    (pin "1")
-  )
   (symbol (lib_id "power:GNDPWR") (at 280.67 107.315 0) (unit 1)
     (in_bom yes) (on_board yes)
@@
     (pin "1")
   )
+  (symbol (lib_id "power:GND") (at 280.67 45.72 0) (unit 1)
+    (in_bom yes) (on_board yes)
+    (property "Reference" "#PWR?" (id 0) (at 280.67 52.07 0)
+      (effects (font (size 1.27 1.27)) hide)
+    )
+    (property "Value" "GND" (id 1) (at 280.797 50.1142 0))
+    (property "Footprint" "" (id 2) (at 280.67 45.72 0)
+      (effects (font (size 1.27 1.27)) hide)
+    )
+    (property "Datasheet" "" (id 3) (at 280.67 45.72 0)
+      (effects (font (size 1.27 1.27)) hide)
+    )
+    (pin "1")
+  )
+  (symbol (lib_id "power:GND") (at 280.67 76.2 0) (unit 1)
+    (in_bom yes) (on_board yes)
+    (property "Reference" "#PWR?" (id 0) (at 280.67 82.55 0)
+      (effects (font (size 1.27 1.27)) hide)
+    )
+    (property "Value" "GND" (id 1) (at 280.797 80.5942 0))
+    (property "Footprint" "" (id 2) (at 280.67 76.2 0)
+      (effects (font (size 1.27 1.27)) hide)
+    )
+    (property "Datasheet" "" (id 3) (at 280.67 76.2 0)
+      (effects (font (size 1.27 1.27)) hide)
+    )
+    (pin "1")
+  )
   (symbol (lib_id "power:GND") (at 334.645 54.61 0) (unit 1)
     (in_bom yes) (on_board yes)
@@
       (effects (font (size 0.762 0.762)))
     )
-    (property "Footprint" "acheron_Components:D_SOD-123_Bidirectional" (id 2) (at 88.265 50.8 0)
+    (property "Footprint" "AcheronComponents:D_SOD-123_Bidirectional" (id 2) (at 88.265 50.8 0)
       (effects (font (size 1.27 1.27)) hide)
     )
@@
       (reference "#PWR0121") (unit 1) (value "GND") (footprint "")
     )
-    (path "/1d0e65fc-efe8-4adc-9ac9-a084bb117e38"
-      (reference "#PWR0122") (unit 1) (value "GNDPWR") (footprint "")
-    )
     (path "/74b05f24-510d-47d9-bb20-f4aad7099401"
       (reference "#PWR0123") (unit 1) (value "GNDPWR") (footprint "")
@@
       (reference "#PWR0164") (unit 1) (value "VCC") (footprint "")
     )
-    (path "/815d9f51-7c0c-4db2-bfe9-68622f963959"
-      (reference "#PWR0165") (unit 1) (value "GNDPWR") (footprint "")
-    )
     (path "/7e5d8d98-24df-4063-a6aa-3f560a47e9e8"
       (reference "#PWR0166") (unit 1) (value "VCC") (footprint "")
@@
       (reference "#PWR0168") (unit 1) (value "VBUS") (footprint "")
     )
+    (path "/65823701-728b-4f18-a87f-22ad8b1ea186"
+      (reference "#PWR?") (unit 1) (value "GND") (footprint "")
+    )
+    (path "/fc70c73c-0303-423d-bfc7-51acb8f8e857"
+      (reference "#PWR?") (unit 1) (value "GND") (footprint "")
+    )
     (path "/47863fa3-1e6f-4aa3-adf2-548a6c2ce974"
       (reference "C1") (unit 1) (value "10u") (footprint "Capacitor_SMD:C_0805_2012Metric_Pad1.15x1.40mm_HandSolder")
@@
     )
     (path "/02ee5b30-d460-4fcb-a6c5-295304092f86"
-      (reference "D1") (unit 1) (value "SMF9.0CA") (footprint "acheron_Components:D_SOD-123_Bidirectional")
+      (reference "D1") (unit 1) (value "SMF9.0CA") (footprint "AcheronComponents:D_SOD-123_Bidirectional")
     )
     (path "/917df597-638e-446e-bec6-35ace98bd373"

Commit message: Initial revision
Parts:
- removed C14, C15, C16, C17: 100nF, Capacitor_SMD:C_0603_1608Metric_Pad1.05x0.95mm_HandSolder, symbol Device:C
Connections:
- net GND: now also U6.2 (GND), U7.2 (GND)
- net GNDPWR: no longer U6.2 (GND), U7.2 (GND)
